File: EAGLE/Controller V1.0.sch (EAGLE design)
At the start: 47 parts, among them IC1 TPS77033, IC2 TPS77033, J2 USB-MICROB, T3 MMBT3906LT1SMD, U1 ATMEGA328P_TQFP, U2 MCP73831, Y1 16MHz

Commit message: h
Parts:
- removed R12, R13, R4: 0, SparkFun-Resistors:0OHM-0603-1/10W-5%
- added TP2: TEST-POINT3X5, SparkFun-Connectors:TEST-POINT3X5
- JP2: device pinhead:PINHD-1X4/90 -> pinhead:PINHD-1X4
Connections:
- new net CAM_GND: C11.2, JP2.4
- new net OLED_GND: C12.2, JP1.1
- net AGND: no longer R13.2
- net GND: no longer C11.2, C12.2, JP1.10, JP2.4, R12.1, R13.1, R4.1
- net GND1: no longer R12.2
- net GND2: no longer R4.2
- net N$13: now also TP2.1
- net OLED_DC: now also JP1.6; no longer JP1.5
- net OLED_MOSI: now also JP1.8; no longer JP1.3
- net OLED_OC: now also JP1.4; no longer JP1.7
- net OLED_RESET: now also JP1.5; no longer JP1.6
- net OLED_SCK: now also JP1.7; no longer JP1.4
- net OLED_VCC: now also JP1.2; no longer JP1.9
Other:
- note added: "0"
- note added: "Group 17"
- note added: "Thermal Imaging HUD Power Distribution and Protection Circuit"
